Commit message: Update AUTODESK.xacro

File: AUTODESK_description/urdf/AUTODESK.xacro (robot description, xacro)
@@ -68,5 +68,5 @@
   <parent link="base_link"/>
   <child link="LEFT_WHEEL_1"/>
-  <axis xyz="-0.0 -1.0 -0.0"/>
+  <axis xyz="0.0 1.0 0.0"/>
 </joint>
 <joint name="Rev2" type="continuous">
